File: power_management.kicad_sch (KiCad schematic)
At the start: 11 parts, among them U401 XC6220B331MR-G, U402 MT3608L

Commit message: update LCSC parts and footprints
Parts:
- L401: footprint Inductor_SMD:L_6.0x6.0_H4.5 -> User Custom Footprint:L_6.0x6.0_H4.5
Changed lines of the file:
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@@
       (effects (font (size 1.27 1.27)))
     )
-    (property "Footprint" "Inductor_SMD:L_6.0x6.0_H4.5" (at 114.3 31.75 0)
+    (property "Footprint" "User Custom Footprint:L_6.0x6.0_H4.5" (at 114.3 31.75 0)
       (effects (font (size 1.27 1.27)) hide)
     )
