File: usbc-2-0.kicad_sch (KiCad schematic)
At the start: 9 parts

Commit message: revise schematics
Parts:
- added D?: SP0503BAHT, Package_TO_SOT_SMD:SOT-143, symbol Power_Protection:SP0503BAHT
- added J?: USB_C_Receptacle_USB2.0, User Custom Footprint:USB_C_Receptable_918-418K2023S40001, symbol Connector:USB_C_Receptacle_USB2.0
- added R? (x2): 5K1, Capacitor_SMD:C_0603_1608Metric, symbol Device:R_Small
Connections:
- net GND: now also D?.1 (A), J?.A1 (GND), J?.A12 (GND), J?.B1 (GND), J?.B12 (GND), J?.S1 (SHIELD), R?.1, R?.1
- net USB_VCC: now reaches D?.4 (K), F?.1, J?.A4 (VBUS), J?.A9 (VBUS), J?.B4 (VBUS), J?.B9 (VBUS)
- net USB_VCC: now also D?.4 (K), J?.A4 (VBUS), J?.A9 (VBUS), J?.B4 (VBUS), J?.B9 (VBUS)
- net ~{PWR_STATUS} renamed ~{PWR}
- new net: J?.A5 (CC1), R?.2
- new net: J?.B5 (CC2), R?.2
- new net D2_N: D?.3 (K), J?.A7 (D-), J?.B7 (D-)
- new net D2_P: D?.2 (K), J?.A6 (D+), J?.B6 (D+)
- no-connect marks 2 -> 4
Other:
- moved on the sheet: Q?
