File: iot_playground.kicad_sch (KiCad schematic)
At the start: 49 parts, among them J101 Micro_SD_Card_Det_Hirose_DM3C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, J102 Conn_01x04, J103 Conn_01x04, J105 Conn_01x02, J701 Conn_01x08, SW101 SW_SPST, SW102 SW_SPST, U101 LIS2DW12, U102 ESP32-WROOM-32E, U103 SHT30-DIS-B2.5KS, U104 LTR-F216A, U105 UHE4913, U106 PCF8563T, Y101 32.768k

Commit message: revise schematics
Parts:
- added C115, C116: 100nF, Capacitor_SMD:C_0603_1608Metric, symbol Device:C_Small
- added H101, H102, H103, H104: MountingHole_Pad, MountingHole:MountingHole_3.2mm_M3_Pad, symbol Mechanical:MountingHole_Pad
- added J701: Conn_01x08, Connector_PinSocket_2.54mm:PinSocket_1x08_P2.54mm_Vertical, symbol Connector_Generic:Conn_01x08
- C103: value 100nF -> 1uF; LCSC C14663 -> (none)
- C108: value 22uF -> 10uF; LCSC C59461 -> (none)
- J105: footprint Connector_JST:JST_PH_B2B-PH-K_1x02_P2.00mm_Vertical -> Connector_JST:JST_PH_S2B-PH-K_1x02_P2.00mm_Horizontal
- U102: value ESP32-WROOM-32E -> ESP32-S3-WROOM-1-N8R2; footprint RF_Module:ESP32-WROOM-32D -> User Custom Footprint:ESP32-S3-WROOM; symbol RF_Module:ESP32-WROOM-32D -> User Symbols:ESP32-S3-WROOM-1-N4R2; LCSC C701341 -> C2913204; MANUFACTURER (none) -> Espressif; MAXIMUM_PACKAGE_HEIGHT (none) -> 3.25mm; PARTREV (none) -> v1.0; STANDARD (none) -> Manufacturer Recommendations
Connections:
- net +5V: now also J701.1 (Pin_1); no longer J701.3 (Pin_3)
- net ACC_INT: now also U102.34 (IO41); no longer U102.12 (IO27)
- net ALS_INT: now also U102.35 (IO42); no longer U102.8 (IO32)
- net EN: now also C115.1
- net ESP_RX: now also U102.36 (IO44/RXD0); no longer U102.34 (RXD0/IO3)
- net ESP_TX: now also U102.37 (IO43/TXD0); no longer U102.35 (TXD0/IO1)
- net GND: now also J701.3 (Pin_3), U102.40 (GND), U102.41_1 (GND), U102.41_2 (GND), U102.41_3 (GND), U102.41_4 (GND), U102.41_5 (GND), U102.41_6 (GND), U102.41_7 (GND), U102.41_8 (GND), U102.41_9 (GND), C115.2, C116.2; no longer J701.4 (Pin_4), J701.5 (Pin_5), U102.15 (GND), U102.38 (GND), U102.39 (GND)
- net HALL_SNSR: now also U102.33 (IO40); no longer U102.23 (IO15)
- net IO0: now also U102.27 (IO0*), C116.1; no longer U102.25 (IO0)
- net IO2: now also U102.38 (IO2), J701.2 (Pin_2); no longer J701.1 (Pin_1), U102.24 (IO2)
- net IO35: now also J701.4 (Pin_4), U102.28 (^IO35); no longer J701.8 (Pin_8), U102.7 (IO35)
- net IO_INT: now also U102.32 (IO39); no longer U102.13 (IO14)
- net LED_IC: now also U102.23 (IO21); no longer U102.14 (IO12)
- net PWR_FLG: now also U102.8 (IO15/XTAL+); no longer U102.26 (IO4)
- net RTC_CLKO: now also J701.8 (Pin_8); no longer J701.6 (Pin_6)
- net RXD1: now also U102.11 (RXD1/IO18); no longer U102.27 (IO16)
- net SD_DET: now also U102.24 (IO47); no longer U102.10 (IO25)
- net SD_MISO: now also U102.22 (IO14); no longer U102.31 (IO19)
- net SD_MOSI: now also U102.21 (IO13); no longer U102.37 (IO23)
- net SD_SCK: now also U102.20 (IO12); no longer U102.30 (IO18)
- net SD_SS: now also U102.19 (IO11); no longer U102.29 (IO5)
- net TXD1: now also U102.10 (TXD1/IO17); no longer U102.28 (IO17)
- net ~{ALRT}: now also U102.9 (IO16/XTAL-); no longer U102.11 (IO26)
- net ~{BUF_EN}: now also U102.31 (IO38); no longer U102.16 (IO13)
- net ~{RTC_INT}: now also U102.25 (IO48); no longer U102.9 (IO33)
- net ~{SCL}: now also U102.18 (IO10); no longer U102.36 (IO22)
- net ~{SDA}: now also U102.17 (IO9); no longer U102.33 (IO21)
- net IO4: now reaches U102.4 (IO4)
- net IO4: now also J701.4 (Pin_4)
- net IO5: now reaches U102.5 (IO5)
- net IO5: now also J701.5 (Pin_5)
- net IO34 renamed IO45
- net IO45: now also U102.26 (*IO45); no longer U102.6 (IO34)
- new net IO1: J701.1 (Pin_1), U102.39 (IO1)
- new net IO3: J701.3 (Pin_3), U102.15 (IO3*)
- new net IO36: J701.5 (Pin_5), U102.29 (^IO36)
- new net IO37: J701.6 (Pin_6), U102.30 (^IO37)
- new net IO6: J701.6 (Pin_6), U102.6 (IO6)
- new net IO7: J701.7 (Pin_7), U102.7 (IO7)
- new net IO8: J701.8 (Pin_8), U102.12 (IO8)
- new net USB_N: U102.13 (D-/IO19)
- new net USB_P: U102.14 (D+/IO20)
- no-connect marks 12 -> 9
Other:
- sheet USBC-2.0 ports: added D2_N, D2_P, ~{PWR}; removed ~{PWR_STATUS}
- note added: "* Strapping pins ^ Octal SPI uses these pins"
- note added: "Analog GPIO Pins Connector"
- note added: "Batteries"
- note added: "Digital GPIO Pins Connector"
- note added: "ESP32-S3-WROOM-1-8NR2"
- note added: "Mounting Holes"
- note removed: "By-pass Caps Pin 2"
- note removed: "ESP32-WROOM-D"
- note removed: "GPIO Pin Connector"
- moved on the sheet: BT101, C103, C108, C109, J102, J105, LED101, LED102, LED103, LED104, LED105, R101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

Commit message: update pcb layout
Other:
- moved on the sheet: C110, C111, U104
